File: T00RA0/Design/T00RA0.brd (EAGLE design)
At the start: 30 x 8.7 mm, 2 parts, among them J1 SM06B-GHS-TB, P1 HEXABIT_17.32_TRIG_P1_P6

Commit message: Fix DRC Generate output Release V0
Routing:
- net P6U: track 7.43 -> 6.44 mm
Other:
- board text added: "P6D"
- board text removed: "TX6"
Changed lines of the file:
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@@
 <text x="33.867853125" y="28.739084375" size="0.8128" layer="26" rot="MR90">3V3</text>
 <text x="30.851603125" y="30.664146875" size="0.8128" layer="26" rot="MR270">P6U</text>
-<text x="29.636209375" y="30.659328125" size="0.8128" layer="26" rot="MR270">TX6</text>
+<text x="29.636209375" y="30.659328125" size="0.8128" layer="26" rot="MR270">P6D</text>
 <text x="32.167075" y="30.6791375" size="0.8128" layer="26" rot="MR270">P1D</text>
 <text x="33.372296875" y="30.676340625" size="0.8128" layer="26" rot="MR270">P1U</text>
@@
 <wire x1="36.3733" y1="30.394903125" x2="36.378134375" y2="30.3997375" width="0.6096" layer="1"/>
 <via x="36.378134375" y="30.3997375" extent="1-16" drill="0.35"/>
-<wire x1="37.374225" y1="27.044903125" x2="36.500975" y2="26.171653125" width="0.6096" layer="1"/>
-<wire x1="28.297475" y1="26.171653125" x2="27.424225" y2="27.044903125" width="0.6096" layer="1"/>
-<wire x1="36.500975" y1="26.171653125" x2="28.297475" y2="26.171653125" width="0.6096" layer="1"/>
 <via x="30.512765625" y="26.160984375" extent="1-16" drill="0.35"/>
 <via x="34.4337625" y="26.160984375" extent="1-16" drill="0.35"/>
-<wire x1="34.4337625" y1="26.160984375" x2="37.374225" y2="27.044903125" width="0" layer="19" extent="1-1"/>
+<wire x1="36.49030625" y1="26.160984375" x2="34.4337625" y2="26.160984375" width="0.6096" layer="1"/>
+<wire x1="37.374225" y1="27.044903125" x2="36.49030625" y2="26.160984375" width="0.6096" layer="1"/>
+<wire x1="34.4337625" y1="26.160984375" x2="30.512765625" y2="26.160984375" width="0.6096" layer="1"/>
+<wire x1="30.512765625" y1="26.160984375" x2="28.30814375" y2="26.160984375" width="0.6096" layer="1"/>
+<wire x1="28.30814375" y1="26.160984375" x2="27.424225" y2="27.044903125" width="0.6096" layer="1"/>
 </signal>
 <signal name="P6U">
@@
 <contactref element="J1" pad="5"/>
 <wire x1="30.524225" y1="30.394903125" x2="30.524225" y2="29.4503125" width="0.4064" layer="1"/>
-<wire x1="25.214015625" y1="29.15821875" x2="26.2007" y2="29.15821875" width="0.4064" layer="1"/>
 <wire x1="30.524225" y1="29.4503125" x2="30.14929375" y2="29.07538125" width="0.4064" layer="1"/>
 <wire x1="25.296853125" y1="29.07538125" x2="25.214015625" y2="29.15821875" width="0.4064" layer="1"/>
